File: pcb/RP2040_tmp.kicad_sch (KiCad schematic)
At the start: 40 parts, among them J0 USB_C_Receptacle_USB2.0, J1 BREAKDOWN, J2 Conn_01x03_Male, SW0 RESET, SW2 RESET, U2 W25Q128JVS, U3 RP2040, U44 SRV05-4, Y0 12MHZ Crystal

Commit message: updated pcb
Parts:
- added SW?: Flip-schalter, symbol Switch:SW_DPDT_x2
Connections:
- net GND: now also SW?.3 (C)
- net VBUS: now also SW?.2 (B); no longer F0.1
- new net: F0.1, SW?.1 (A)
Other:
- moved on the sheet: F0
Changed lines of the file:
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@@
   (junction (at 175.26 161.798) (diameter 0) (color 0 0 0 0)
   )
+  (junction (at 59.182 110.236) (diameter 0) (color 0 0 0 0)
+  )
   (junction (at 26.162 228.346) (diameter 0) (color 0 0 0 0)
   )
@@
   )
   (junction (at 89.2302 219.3544) (diameter 0) (color 0 0 0 0)
-  )
-  (junction (at 52.1462 122.9106) (diameter 0) (color 0 0 0 0)
   )
   (junction (at 209.55 141.478) (diameter 0) (color 0 0 0 0)
@@
     (stroke (width 0) (type default) (color 0 0 0 0))
   )
-  (wire (pts (xy 52.1462 122.936) (xy 52.1462 122.9106))
+  (wire (pts (xy 59.182 110.2614) (xy 59.182 110.236))
     (stroke (width 0) (type default) (color 0 0 0 0))
   )
@@
     (stroke (width 0) (type default) (color 0 0 0 0))
   )
-  (wire (pts (xy 44.45 122.936) (xy 52.1462 122.936))
-    (stroke (width 0) (type default) (color 0 0 0 0))
-  )
   (polyline (pts (xy 12.7 210.566) (xy 12.7 190.754))
     (stroke (width 0) (type default) (color 0 0 0 0))
@@
     (stroke (width 0) (type default) (color 0 0 0 0))
   )
+  (wire (pts (xy 49.022 122.936) (xy 49.022 112.776))
+    (stroke (width 0) (type default) (color 0 0 0 0))
+  )
   (wire (pts (xy 163.83 151.638) (xy 163.83 150.368))
     (stroke (width 0) (type default) (color 0 0 0 0))
@@
   )
   (wire (pts (xy 84.1248 226.9744) (xy 87.884 226.9744))
+    (stroke (width 0) (type default) (color 0 0 0 0))
+  )
+  (wire (pts (xy 44.45 122.936) (xy 49.022 122.936))
     (stroke (width 0) (type default) (color 0 0 0 0))
   )
@@
     )
   )
+  (global_label "GND" (shape input) (at 59.182 115.316 0) (fields_autoplaced)
+    (effects (font (size 1.27 1.27)) (justify left))
+    (property "Intersheet References" "${INTERSHEET_REFS}" (id 0) (at 65.4656 115.2366 0)
+      (effects (font (size 1.27 1.27)) (justify left) hide)
+    )
+  )
   (global_label "+5V" (shape input) (at 87.376 136.398 90) (fields_autoplaced)
     (effects (font (size 1.27 1.27)) (justify left))
@@
     )
   )
-  (global_label "+5V" (shape input) (at 57.2262 122.9106 0) (fields_autoplaced)
-    (effects (font (size 1.27 1.27)) (justify left))
-    (property "Intersheet References" "${INTERSHEET_REFS}" (id 0) (at 63.5098 122.8312 0)
+  (global_label "+5V" (shape input) (at 64.262 110.236 0) (fields_autoplaced)
+    (effects (font (size 1.27 1.27)) (justify left))
+    (property "Intersheet References" "${INTERSHEET_REFS}" (id 0) (at 70.5456 110.1566 0)
       (effects (font (size 1.27 1.27)) (justify left) hide)
     )
@@
     (pin "1")
   )
-  (symbol (lib_id "Device:Polyfuse_Small") (at 54.6862 122.9106 90) (unit 1)
-    (in_bom yes) (on_board yes)
-    (property "Reference" "F0" (id 0) (at 54.1274 120.5484 90))
-    (property "Value" "polyfuse" (id 1) (at 59.1312 120.3706 90))
-    (property "Footprint" "Fuse:Fuse_1206_3216Metric" (id 2) (at 59.7662 121.6406 0)
-      (effects (font (size 1.27 1.27)) (justify left) hide)
-    )
-    (property "Datasheet" "~" (id 3) (at 54.6862 122.9106 0)
-      (effects (font (size 1.27 1.27)) hide)
-    )
-    (property "LCSC" "C69688" (id 4) (at 54.6862 122.9106 0)
+  (symbol (lib_id "Device:Polyfuse_Small") (at 61.722 110.236 90) (unit 1)
+    (in_bom yes) (on_board yes)
+    (property "Reference" "F0" (id 0) (at 61.1632 107.8738 90))
+    (property "Value" "polyfuse" (id 1) (at 66.167 107.696 90))
+    (property "Footprint" "Fuse:Fuse_1206_3216Metric" (id 2) (at 66.802 108.966 0)
+      (effects (font (size 1.27 1.27)) (justify left) hide)
+    )
+    (property "Datasheet" "~" (id 3) (at 61.722 110.236 0)
+      (effects (font (size 1.27 1.27)) hide)
+    )
+    (property "LCSC" "C69688" (id 4) (at 61.722 110.236 0)
       (effects (font (size 1.27 1.27)) hide)
     )
@@
     (pin "1")
   )
+  (symbol (lib_id "Switch:SW_DPDT_x2") (at 54.102 112.776 0) (unit 1)
+    (in_bom yes) (on_board yes) (fields_autoplaced)
+    (property "Reference" "SW?" (id 0) (at 54.102 104.14 0))
+    (property "Value" "Flip-schalter" (id 1) (at 54.102 106.68 0))
+    (property "Footprint" "" (id 2) (at 54.102 112.776 0)
+      (effects (font (size 1.27 1.27)) hide)
+    )
+    (property "Datasheet" "~" (id 3) (at 54.102 112.776 0)
+      (effects (font (size 1.27 1.27)) hide)
+    )
+    (pin "1")
+    (pin "2")
+    (pin "3")
+    (pin "4")
+    (pin "5")
+    (pin "6")
+  )
   (symbol (lib_id "Power_Protection:SRV05-4") (at 87.376 149.098 0) (unit 1)
     (in_bom yes) (on_board yes) (fields_autoplaced)
@@
       (reference "SW?") (unit 1) (value "RotaryEncoder_Switch") (footprint "")
     )
+    (path "/e177d86e-eaee-4d07-bfea-120b6b4265c0"
+      (reference "SW?") (unit 1) (value "Flip-schalter") (footprint "")
+    )
     (path "/00000000-0000-0000-0000-00005eda5f2c"
